File: schematics/PLD_Controller_Board/PLD Controller Board.sch (EAGLE design)
At the start: 35 parts, among them IC2 ATMEGA328-PU

Commit message: schematic update
Parts:
- added C5: 10uF, SparkFun-Capacitors:10UF-POLAR-RADIAL-2.5MM-25V-20%
- RESET/RX/TX: device pinhead:PINHD-1X3 -> pinhead:PINHD-1X4
Connections:
- net +5V: now also R1-RESET.2; no longer R1-RESET.1
- net GND: now also RESET.S
- net N$1: now also C5.-, R1-RESET.1, RESET.P, RESET/RX/TX.2; no longer RESET.S, RESET/RX/TX.1
- net N$38: now also RESET/RX/TX.3; no longer RESET/RX/TX.2
- net N$39: now also RESET/RX/TX.4; no longer RESET/RX/TX.3
- net N$4: now also C5.+, RESET/RX/TX.1; no longer R1-RESET.2, RESET.P
Other:
- moved on the sheet: R1-RESET, RESET
